File: PCB/ValveController.kicad_pcb (KiCad board)
At the start: 2 copper layers, 50 x 50 mm, 39 parts, among them J1 Conn_01x04, J2 TTP224, J3 Valve 1, J4 Valve 2, J5 Input 24V, J6 4-20 IO, Q1 30N06, Q2 30N06, Q3 2N7002, Q4 AO3401A, Q5 2N7002, Q6 SI2319A, Q7 BC807, U1 ESP32-C3-SuperMini, U2 XTR111AxDGQ, U3 MCP4725xxx-xCH, U4 UMW_78M05_TO252, U5 PCF8574DWR

Commit message: Scheme and PCB updates
Parts:
- C1, C2: value 100nF -> 0.1uF
- C10, C8, C9: value 1nF -> 1uF
- C7: value 10nF -> 0.1uF
- R2: value R -> 50R
- R3, R4: footprint Resistor_SMD:R_0805_2012Metric_Pad1.20x1.40mm_HandSolder -> Capacitor_SMD:C_0603_1608Metric_Pad1.08x0.95mm_HandSolder
- R5: value 3K3 -> 3K
- moved C5 6.77 mm to (61.0, 91.2)
- moved R1 4.07 mm to (59.8, 88.2)
- moved C4 3.58 mm to (75.2, 69.2), turned to 0 degrees
- moved R2 3.02 mm to (70.2, 90.5), turned to -90 degrees
- moved RV1 1.95 mm to (54.8, 82.0)
- moved R3 0.35 mm to (67.8, 71.2)
Routing:
- net GNDPWR: track 229.5 -> 233.5 mm
- net +24V: track 95.0 -> 91.5 mm, vias 3 -> 2
- net /4-20 Input +: track 28.0 -> 25.3 mm
- net Net-(R1-Pad2): track 2.60 -> 4.52 mm
- net Net-(U1-GPIO3): track 20.3 -> 18.5 mm
- net +3.3V: track 135.3 -> 136.2 mm
- net Net-(J1-Pin_3): track 61.3 -> 60.4 mm
