File: PCB/ValveController.kicad_sch (KiCad schematic)
At the start: 39 parts, among them J1 Conn_01x04, J2 TTP224, J3 Valve 1, J4 Valve 2, J5 Input 24V, J6 4-20 IO, Q1 30N06, Q2 30N06, Q3 2N7002, Q4 AO3401A, Q5 2N7002, Q6 SI2319A, Q7 BC807, U1 ESP32-C3-SuperMini, U2 XTR111AxDGQ, U3 MCP4725xxx-xCH, U4 UMW_78M05_TO252, U5 PCF8574DWR

Commit message: Scheme and PCB updates
Parts:
- C1, C2: value 100nF -> 0.1uF
- C10, C8, C9: value 1nF -> 1uF
- C7: value 10nF -> 0.1uF
- R2: value R -> 50R
- R3, R4: footprint Resistor_SMD:R_0805_2012Metric_Pad1.20x1.40mm_HandSolder -> Capacitor_SMD:C_0603_1608Metric_Pad1.08x0.95mm_HandSolder
- R5: value 3K3 -> 3K
Other:
- moved on the sheet: R5
Changed lines of the file:
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@@
 	(paper "A4")
 	(junction
+		(at 57.15 68.58)
+		(diameter 0)
+		(color 0 0 0 0)
+	)
+	(junction
 		(at 233.68 29.21)
 		(diameter 0)
@@
 	)
 	(junction
-		(at 60.96 68.58)
-		(diameter 0)
-		(color 0 0 0 0)
-	)
-	(junction
 		(at 162.56 105.41)
 		(diameter 0)
@@
 	)
 	(junction
-		(at 220.98 111.76)
+		(at 85.09 88.9)
 		(diameter 0)
 		(color 0 0 0 0)
 	)
 	(junction
-		(at 234.95 67.31)
+		(at 220.98 111.76)
 		(diameter 0)
 		(color 0 0 0 0)
 	)
 	(junction
-		(at 50.8 78.74)
+		(at 234.95 67.31)
 		(diameter 0)
 		(color 0 0 0 0)
 	)
 	(junction
-		(at 152.4 76.2)
+		(at 50.8 78.74)
 		(diameter 0)
 		(color 0 0 0 0)
 	)
 	(junction
-		(at 86.36 88.9)
+		(at 152.4 76.2)
 		(diameter 0)
 		(color 0 0 0 0)
 	)
 	(junction
-		(at 86.36 81.28)
+		(at 85.09 81.28)
 		(diameter 0)
 		(color 0 0 0 0)
@@
 	(wire
 		(pts
-			(xy 73.66 88.9) (xy 86.36 88.9)
+			(xy 73.66 88.9) (xy 85.09 88.9)
+		)
+		(stroke
+			(width 0)
+			(type default)
+		)
+	)
+	(wire
+		(pts
+			(xy 85.09 81.28) (xy 88.9 81.28)
 		)
 		(stroke
@@
 	(wire
 		(pts
-			(xy 86.36 88.9) (xy 88.9 88.9)
-		)
-		(stroke
-			(width 0)
-			(type default)
-		)
-	)
-	(wire
-		(pts
 			(xy 73.66 55.88) (xy 73.66 63.5)
 		)
@@
 	(wire
 		(pts
-			(xy 60.96 68.58) (xy 63.5 68.58)
-		)
-		(stroke
-			(width 0)
-			(type default)
-		)
-	)
-	(wire
-		(pts
 			(xy 254 149.86) (xy 254 144.78)
 		)
@@
 	(wire
 		(pts
-			(xy 57.15 68.58) (xy 60.96 68.58)
+			(xy 57.15 68.58) (xy 63.5 68.58)
 		)
 		(stroke
@@
 	(wire
 		(pts
-			(xy 86.36 81.28) (xy 88.9 81.28)
-		)
-		(stroke
-			(width 0)
-			(type default)
-		)
-	)
-	(wire
-		(pts
 			(xy 233.68 29.21) (xy 217.17 29.21)
 		)
@@
 	(wire
 		(pts
+			(xy 57.15 55.88) (xy 60.96 55.88)
+		)
+		(stroke
+			(width 0)
+			(type default)
+		)
+	)
+	(wire
+		(pts
 			(xy 227.33 64.77) (xy 217.17 64.77)
 		)
@@
 	(wire
 		(pts
+			(xy 85.09 88.9) (xy 88.9 88.9)
+		)
+		(stroke
+			(width 0)
+			(type default)
+		)
+	)
+	(wire
+		(pts
 			(xy 27.94 107.95) (xy 34.29 107.95)
 		)
@@
 	(wire
 		(pts
-			(xy 83.82 81.28) (xy 86.36 81.28)
+			(xy 83.82 81.28) (xy 85.09 81.28)
 		)
 		(stroke
@@
 	(wire
 		(pts
-			(xy 60.96 55.88) (xy 60.96 68.58)
+			(xy 57.15 55.88) (xy 57.15 68.58)
 		)
 		(stroke
@@
 		(on_board yes)
 		(dnp no)
-		(fields_autoplaced yes)
 		(property "Reference" "R6"
-			(at 91.44 83.8199 0)
+			(at 89.916 83.82 0)
 			(effects
 				(font
@@
 		)
 		(property "Value" "3K3"
-			(at 91.44 86.3599 0)
+			(at 89.916 86.36 0)
 			(effects
 				(font
@@
 			)
 		)
-		(property "Value" "1nF"
+		(property "Value" "1uF"
 			(at 166.37 100.33 90)
 			(effects
@@
 			)
 		)
-		(property "Value" "R"
+		(property "Value" "50R"
 			(at 236.22 34.2899 0)
 			(effects
@@
 			)
 		)
-		(property "Value" "10nF"
+		(property "Value" "0.1uF"
 			(at 44.45 101.5999 0)
 			(effects
@@
 			)
 		)
-		(property "Value" "1nF"
+		(property "Value" "1uF"
 			(at 106.68 59.69 90)
 			(effects
@@
 			)
 		)
-		(property "Value" "100nF"
+		(property "Value" "0.1uF"
 			(at 231.14 74.9299 0)
 			(effects
@@
 			)
 		)
-		(property "Value" "1nF"
+		(property "Value" "1uF"
 			(at 64.77 50.8 90)
 			(effects
@@
 	(symbol
 		(lib_id "Device:R")
-		(at 86.36 85.09 0)
+		(at 85.09 85.09 0)
 		(unit 1)
 		(exclude_from_sim no)
@@
 		(on_board yes)
 		(dnp no)
-		(fields_autoplaced yes)
 		(property "Reference" "R5"
-			(at 88.9 83.8199 0)
+			(at 83.82 83.82 0)
 			(effects
 				(font
@@
 			)
 		)
-		(property "Value" "3K3"
-			(at 88.9 86.3599 0)
+		(property "Value" "3K"
+			(at 83.82 86.36 0)
 			(effects
 				(font
@@
 		)
 		(property "Footprint" "Capacitor_SMD:C_0603_1608Metric_Pad1.08x0.95mm_HandSolder"
-			(at 84.582 85.09 90)
+			(at 83.312 85.09 90)
 			(effects
 				(font
@@
 		)
 		(property "Datasheet" "~"
-			(at 86.36 85.09 0)
+			(at 85.09 85.09 0)
 			(effects
 				(font
@@
 		)
 		(property "Description" "Resistor"
-			(at 86.36 85.09 0)
+			(at 85.09 85.09 0)
 			(effects
 				(font
@@
 			)
 		)
-		(property "Footprint" "Resistor_SMD:R_0805_2012Metric_Pad1.20x1.40mm_HandSolder"
+		(property "Footprint" "Capacitor_SMD:C_0603_1608Metric_Pad1.08x0.95mm_HandSolder"
 			(at 163.322 67.31 90)
 			(effects
@@
 			)
 		)
-		(property "Footprint" "Resistor_SMD:R_0805_2012Metric_Pad1.20x1.40mm_HandSolder"
+		(property "Footprint" "Capacitor_SMD:C_0603_1608Metric_Pad1.08x0.95mm_HandSolder"
 			(at 156.972 67.31 90)
 			(effects
@@
 			)
 		)
-		(property "Value" "100nF"
+		(property "Value" "0.1uF"
 			(at 238.76 74.9299 0)
 			(effects

Commit message: refactoring
Parts:
- RV1: footprint Connector_JST:JST_XH_B3B-XH-A_1x03_P2.50mm_Vertical -> Connector_Wire:SolderWire-0.5sqmm_1x03_P4.6mm_D0.9mm_OD2.1mm
Connections:
- net I2C_SDA: now reaches J1.4 (Pin_4), R4.2, U1.12 (GPIO8), U3.4 (SDA), U5.15 (SDA)
- net I2C_SCL: now reaches J1.3 (Pin_3), R3.2, U1.13 (GPIO9), U3.5 (SCL), U5.14 (SCL)
Changed lines of the file:
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@@
 		)
 	)
+	(label "I2C_SCL"
+		(at 152.4 91.44 0)
+		(effects
+			(font
+				(size 1.27 1.27)
+			)
+			(justify left bottom)
+		)
+	)
+	(label "I2C_SDA"
+		(at 149.86 88.9 0)
+		(effects
+			(font
+				(size 1.27 1.27)
+			)
+			(justify left bottom)
+		)
+	)
 	(label "4-20 Input +"
 		(at 31.75 121.92 0)
@@
 			)
 		)
-		(property "Footprint" "Connector_JST:JST_XH_B3B-XH-A_1x03_P2.50mm_Vertical"
+		(property "Footprint" "Connector_Wire:SolderWire-0.5sqmm_1x03_P4.6mm_D0.9mm_OD2.1mm"
 			(at 256.54 74.93 0)
 			(effects
